Commit message: Imported upstream version '1.0.2' of 'upstream'

File: webots_ros2_ur_e_description/urdf/ur5e_robot.urdf (robot description, URDF)
Before this commit: robot ur5e, 7 links, 6 joints
Links:
- added link base
- added link ee_link; collision box size=0.01 0.01 0.01
- added link tool0
- added link world
Joints:
- added joint base_link-base_fixed_joint: type fixed, parent base_link, child base, origin xyz=0 0 0 rpy=0 0 -3.141592653589793
- added joint ee_fixed_joint: type fixed, parent wrist_3_link, child ee_link, origin xyz=0.0 0.1 0.0 rpy=0.0 0.0 1.5707963267948966
- added joint world_joint: type fixed, parent world, child base_link, origin xyz=0.0 0.0 0.0 rpy=0.0 0.0 0.0
- added joint wrist_3_link-tool0_fixed_joint: type fixed, parent wrist_3_link, child tool0, origin xyz=0 0.1 0 rpy=-1.5707963267948966 0 0

Commit message: Rebase from 'upstream'

File: webots_ros2_ur_e_description/urdf/ur5e_robot.urdf (robot description, URDF)
Before this commit: robot ur5e, 11 links, 10 joints
Links:
- removed link base
- removed link ee_link
- removed link tool0
- removed link world
Joints:
- removed joint base_link-base_fixed_joint
- removed joint ee_fixed_joint
- removed joint world_joint
- removed joint wrist_3_link-tool0_fixed_joint
